Commit message: Updated urdf_from_xacro

File: navvis_description/urdf/robot.xacro (robot description, xacro)
@@ -3,5 +3,5 @@
     <link name="base">
         <visual>
-        <!-- Shift the box up half its height. !-->
+            <!-- Shift the box up half its height. !-->
             <origin xyz="0.0 0.0 0.96" rpy="0.0 0.0 0.0" />
             <geometry>
@@ -10,5 +10,5 @@
         </visual>
         <collision>
-        <!-- Shift the box up half its height. !-->
+            <!-- Shift the box up half its height. !-->
             <origin xyz="0.0 0.0 0.96" rpy="0.0 0.0 0.0" />
             <geometry>
@@ -17,9 +17,4 @@
         </collision>
     </link>
-    <joint name="base_laser_vert_bottom_joint" type="fixed">
-        <parent link="base" />
-        <child link="laser_vert_bottom" />
-        <origin xyz="0.3158 -0.0021 0.5100" rpy="3.1355 -1.3045 0.0025" />
-    </joint>
     <!-- XACRO Macro definition block to add around the wheel link and joint !-->
     <xacro:macro name="xacro_name" params="side reflect">
@@ -33,5 +28,5 @@
                 <origin xyz="0.0 0.0 0.0" rpy="0.0 0.0 0.0" />
                 <geometry>
-                    <cylinder radius="0.2" length="0.05"/>
+                    <cylinder radius="0.2" length="0.05" />
                 </geometry>
             </visual>
@@ -39,5 +34,5 @@
                 <origin xyz="0.0 0.0 0.0" rpy="0.0 0.0 0.0" />
                 <geometry>
-                    <cylinder radius="0.2" length="0.05"/>
+                    <cylinder radius="0.2" length="0.05" />
                 </geometry>
             </collision>
@@ -51,24 +46,10 @@
         <child link="wheel_center" />
         <origin xyz="0.1 0 0" rpy="${-pi/2} 0 0" />
-     </joint>
-     <link name="wheel_center">
-         <visual>
-	    <origin xyz="0.0 0.0 0.0" rpy="0.0 0.0 0.0" />
-	    <geometry>
-	        <cylinder radius="0.15" length="0.05"/>
-	    </geometry>
-        </visual>
-        <collision>
-	    <origin xyz="0.0 0.0 0.0" rpy="0.0 0.0 0.0" />
-	    <geometry>
-	        <cylinder radius="0.15" length="0.05"/>
-	    </geometry>
-        </collision>
-    </link>
-    <link name="laser_vert_bottom">
+    </joint>
+    <link name="wheel_center">
         <visual>
             <origin xyz="0.0 0.0 0.0" rpy="0.0 0.0 0.0" />
             <geometry>
-                <box size="0.62 0.62 0.87" />
+                <cylinder radius="0.15" length="0.05" />
             </geometry>
         </visual>
@@ -76,76 +57,28 @@
             <origin xyz="0.0 0.0 0.0" rpy="0.0 0.0 0.0" />
             <geometry>
-                <box size="0.62 0.62 0.87" />
-            </geometry>
-        </collision>
-    </link>
-    <joint name="laser_vert_top_right_joint" type="fixed">
-        <parent link="base" />
-        <child link="laser_vert_top_right" />
-        <origin xyz="0.2978 -0.145 1.8451" rpy="-1.8451 0.6313 -1.9377" />
-    </joint>
-    <link name="laser_vert_top_right">
-        <visual>
-            <origin xyz="0.0 0.0 0.0" rpy="0.0 0.0 0.0" />
-            <geometry>
-                <box size="0.62 0.62 0.87" />
-            </geometry>
-        </visual>
-        <collision>
-            <origin xyz="0.0 0.0 0.0" rpy="0.0 0.0 0.0" />
-            <geometry>
-                <box size="0.62 0.62 0.87" />
-            </geometry>
-        </collision>
-    </link>
-    <joint name="laser_vert_top_left_joint" type="fixed">
-        <parent link="base" />
-        <child link="laser_vert_top_left" />
-        <origin xyz="0.2997 0.1531 1.8443" rpy="1.1780 0.6198 1.9560" />
-    </joint>
-    <link name="laser_vert_top_left">
-        <visual>
-            <origin xyz="0.0 0.0 0.0" rpy="0.0 0.0 0.0" />
-            <geometry>
-                <box size="0.62 0.62 0.87" />
-            </geometry>
-        </visual>
-        <collision>
-            <origin xyz="0.0 0.0 0.0" rpy="0.0 0.0 0.0" />
-            <geometry>
-                <box size="0.62 0.62 0.87" />
-            </geometry>
-        </collision>
-    </link>
-    <joint name="laser_horiz_joint" type="fixed">
-        <parent link="base" />
-        <child link="laser_horiz" />
-        <origin xyz="0.2325 0.0001 1.9201" rpy="-0.00120 0.1146 -0.0015" />
-    </joint>
-    <link name="laser_horiz">
-        <visual>
-            <origin xyz="0.0 0.0 0.0" rpy="0.0 0.0 0.0" />
-            <geometry>
-                <cylinder radius="0.52" length="0.72"/>
-            </geometry>
-        </visual>
-        <collision>
-            <origin xyz="0.0 0.0 0.0" rpy="0.0 0.0 0.0" />
-            <geometry>
-                <cylinder radius="0.52" length="0.72"/>
+                <cylinder radius="0.15" length="0.05" />
             </geometry>
         </collision>
     </link>
     <!-- Include the XACRO file that defines a Hokuyo LIDAR. -->
-    <xacro:include filename="$(find gazebo_plugins)/test/multi_robot_scenario/xacro/laser/hokuyo.xacro" />
-    <xacro:laser name="laser_vert_bottom" parent="base" xyz="0.3157894464801903 -0.002068548615034871 0.5099999434059285" rpy="3.1354753 -1.3045001 0.0024658"
-meshes="package://gazebo_plugins/test/multi_robot_scenario/meshes/laser" />
-    <xacro:laser name="laser_vert_top_left" parent="base" xyz="0.2997 0.1531 1.8443" rpy="1.780 0.6198 1.9560" meshes="package://gazebo_plugins/test/multi_robot_scenario/meshes/laser" />
-    <xacro:laser name="laser_vert_top_right" parent="base" xyz="0.2978 -0.1450 1.8451" rpy="-1.1760 0.6313 -1.9377" meshes="package://gazebo_plugins/test/multi_robot_scenario/meshes/laser" />
+    <xacro:include
+        filename="$(find gazebo_plugins)/test/multi_robot_scenario/xacro/laser/hokuyo.xacro" />
+    <xacro:laser name="laser_vert_bottom" parent="base"
+        xyz="0.3157894464801903 -0.002068548615034871 0.5099999434059285"
+        rpy="3.1354753 -1.3045001 0.0024658"
+        meshes="package://gazebo_plugins/test/multi_robot_scenario/meshes/laser" />
+    <xacro:laser name="laser_vert_top_left" parent="base" xyz="0.2997 0.1531 1.8443"
+        rpy="1.780 0.6198 1.9560"
+        meshes="package://gazebo_plugins/test/multi_robot_scenario/meshes/laser" />
+    <xacro:laser name="laser_vert_top_right" parent="base" xyz="0.2978 -0.1450 1.8451"
+        rpy="-1.1760 0.6313 -1.9377"
+        meshes="package://gazebo_plugins/test/multi_robot_scenario/meshes/laser" />
     <!-- Include the XACRO file that defines a Hokuyo LIDAR. -->
-    <xacro:include filename="$(find velodyne_description)/urdf/VLP-16.urdf.xacro"/>
+    <xacro:include filename="$(find velodyne_description)/urdf/VLP-16.urdf.xacro" />
     <!-- Invoke the macro to define the Hokuyo LIDAR. -->
-    <xacro:VLP-16 parent="base" name="laser_horiz" topic="laser_horiz/packets" hz="10" samples="440" gpu="false">
-        <origin xyz="0.2325416305773505 -0.0001380069427607134 1.920122926231907" rpy="-0.0012068 0.114646 -0.0015308" />
+    <xacro:VLP-16 parent="base" name="laser_horiz" topic="laser_horiz/packets" hz="10" samples="440"
+        gpu="false">
+        <origin xyz="0.2325416305773505 -0.0001380069427607134 1.920122926231907"
+            rpy="-0.0012068 0.114646 -0.0015308" />
     </xacro:VLP-16>
 </robot>
